Commit message: Boh non si capisce urdf

File: urdf/robot4.xacro (robot description, xacro)
@@ -115,7 +115,59 @@
     <joint_properties damping="1.0" friction="1.0"/>
   </joint>
+  <!--arm definition -->
+  <link name="arm_base_link">
+  	<inertial>
+  		<mass value="0.1"/>
+  		<origin xyz="0 0 0" rpy="0 0 0" />
+  		<inertia ixx="0.0000416666667" ixy="0" ixz="0" iyy="0.0000416666667" iyz="0" izz="0.0000416666667"/>
+  	</inertial>
+  	<collision>
+  	  <origin xyz="0 0 0" rpy="0 0 0"/>
+      <geometry>
+        <box size="0.1 0.1 0.1"/>
+      </geometry>
+  	</collision>
+  	<visual>
+  	  <origin xyz="0 0 0" rpy="0 0 0"/>
+      <geometry>
+        <box size="0.1 0.1 0.1"/>
+      </geometry>
+      <material name="red" />
+  	</visual>
+  </link>
+  <joint name="arm_base_to_base" type="fixed">
+  	<origin rpy="0 0 0" xyz="0 0 0.085"/>
+  	<parent link="link_chassis"/>
+  	<child link="arm_base_link"/>
+  </joint>
+  <link name="arm_link_01">
+  	<inertial>
+  		<mass value="0.025"/>
+  		<origin xyz="0 0 0" rpy="0 0 0" />
+  		<inertia ixx="0.000010279" ixy="0" ixz="0" iyy="0.000010279" iyz="0" izz="0.000007225"/>
+  	</inertial>
+  	<collision>
+  	  <origin xyz="0 0 0" rpy="0 0 0"/>
+      <geometry>
+        <cylinder radius="0.04" length="0.08"/>
+      </geometry>
+  	</collision>
+  	<visual>
+  	  <origin xyz="0 0 0" rpy="0 0 0"/>
+      <geometry>
+        <cylinder radius="0.04" length="0.08"/>
+      </geometry>
+      <material name="red" />
+  	</visual>
+  </link>
+  <joint name="arm_joint_01" type="continuous">
+  	<axis xyz="0 0 1"/>
+  	<origin rpy="0 0 0" xyz="0 0 0.09"/>
+  	<parent link="arm_base_link"/>
+  	<child link="arm_link_01"/>
+  </joint>
   <link name="camera_link">
 	    <collision>
-	      <origin xyz="0 0 0.025" rpy="0 0 0"/>
+	      <origin xyz="0 0 0.06" rpy="0 0 0"/>
 	      <geometry>
 		<box size="0.05 0.05 0.05"/>
@@ -123,5 +175,5 @@
 	    </collision>
 	    <visual>
-	      <origin xyz="0 0 0.025" rpy="0 0 0"/>
+	      <origin xyz="0 0 0.06" rpy="0 0 0"/>
 	      <geometry>
 		<box size="0.05 0.05 0.05"/>
@@ -139,6 +191,6 @@
   <joint name="camera_joint" type="fixed">
 	    <axis xyz="0 1 0" />
-	    <origin xyz="0.23 0 0.0" rpy="0 0 0"/>
-	    <parent link="link_chassis"/>
+	    <origin xyz="0.0 0 0.0" rpy="0 0 0"/>
+	    <parent link="arm_link_01"/>
 	    <child link="camera_link"/>
 	 </joint>

Commit message: ultimo commit qui

File: urdf/robot4.xacro (robot description, xacro)
@@ -1,44 +1,56 @@
 <?xml version="1.0"?>
 <robot xmlns:xacro="http://www.ros.org/wiki/xacro" name="robot4_xacro">
-<xacro:include filename="$(find robot_urdf)/urdf/robot4.gazebo"/>
-	<xacro:property name="length_wheel" value="0.04" />
+ <xacro:include filename="$(find robot_urdf)/urdf/robot4.gazebo"/>
+ <xacro:include filename="$(find robot_urdf)/urdf/materials.xacro" />
+  <!-- Inertia definition (cylinder, wheel + chassis) -->
+  <xacro:macro name="cylinder_inertia" params="mass r l">
+    <inertia ixx="${mass*(3*r*r+l*l)/12}" ixy = "0" ixz = "0"
+                iyy="${mass*(3*r*r+l*l)/12}" iyz = "0" izz="${mass*(r*r)/2}" />
+  </xacro:macro>
+	<xacro:macro name="default_inertial" params="mass">
+      <inertial>
+        <mass value="${mass}" />
+        <origin rpy="0 1.5707 1.5707" xyz="0 0 0"/>
+        <inertia ixx="0.000526666666667" ixy="0" ixz="0" iyy="0.000526666666667" iyz="0" izz="0.001"/>
+      </inertial>
+	</xacro:macro>
+  <!-- Wheel defnition -->
+  <xacro:property name="length_wheel" value="0.04" />
 	<xacro:property name="radius_wheel" value="0.1" />
-	<xacro:macro name="default_inertial" params="mass">
-               <inertial>
-                       <mass value="${mass}" />
-                       <origin rpy="0 1.5707 1.5707" xyz="0 0 0"/>
-                       <inertia ixx="0.000526666666667" ixy="0" ixz="0" iyy="0.000526666666667" iyz="0" izz="0.001"/>
-               </inertial>
-	</xacro:macro>
-    <xacro:macro name="wheel_geometry">
+  <xacro:property name="mass_wheel" value="0.2" />
+  <!-- geometry-->
+  <xacro:macro name="wheel_geometry">
 		<geometry>
        			<cylinder length="${length_wheel}" radius="${radius_wheel}"/>
      	</geometry>
 	</xacro:macro>
-  <material name="black">
-    <color rgba="0.0 0.0 0.0 1.0"/>
-  </material>
-  <material name="blue">
-    <color rgba="0.203125 0.23828125 0.28515625 1.0"/>
-  </material>
-  <material name="green">
-    <color rgba="0.0 0.8 0.0 1.0"/>
-  </material>
-  <material name="grey">
-    <color rgba="0.2 0.2 0.2 1.0"/>
-  </material>
-  <material name="orange">
-    <color rgba="1.0 0.423529411765 0.0392156862745 1.0"/>
-  </material>
-  <material name="brown">
-    <color rgba="0.870588235294 0.811764705882 0.764705882353 1.0"/>
-  </material>
-  <material name="red">
-    <color rgba="0.80078125 0.12890625 0.1328125 1.0"/>
-  </material>
-  <material name="white">
-    <color rgba="1.0 1.0 1.0 1.0"/>
-  </material>
-	  <link name="link_chassis">
+  <!-- link -->
+  <xacro:macro name="link_wheel" params="name">
+    <link name="${name}">
+        <xacro:default_inertial mass="${mass_wheel}"/>
+        <collision name="${name}_collision">
+          <origin rpy="0 1.5707 1.5707" xyz="0 0 0"/>
+          <xacro:wheel_geometry />
+        </collision>
+        <visual name="${name}_visual">
+          <origin rpy="0 1.5707 1.5707" xyz="0 0 0"/>
+          <xacro:wheel_geometry />
+          <material name="red"/>
+        </visual>
+    </link>
+  </xacro:macro>
+  <!-- joint -->
+  <xacro:macro name="joint_wheel" params="name child origin_xyz">
+    <joint name="${name}" type="continuous">
+      <origin rpy="0 0 0" xyz="${origin_xyz}"/>
+      <child link="${child}"/>
+      <parent link="link_chassis"/>
+      <axis rpy="0 0 0" xyz="0 1 0"/>
+      <limit effort="10000" velocity="1000"/>
+      <joint_properties damping="1.0" friction="1.0"/>
+    </joint>
+  </xacro:macro>
+  <!-- Chassis definition -->
+  <link name="link_chassis">
     <!-- pose and inertial -->
     <pose>0 0 0.1 0 0 0</pose>
@@ -75,44 +87,9 @@
     </visual>
   </link>
-   <link name="link_right_wheel">
-    <xacro:default_inertial mass="0.2"/>
-    <collision name="link_right_wheel_collision">
-      <origin rpy="0 1.5707 1.5707" xyz="0 0 0"/>
-      <xacro:wheel_geometry />
-    </collision>
-    <visual name="link_right_wheel_visual">
-      <origin rpy="0 1.5707 1.5707" xyz="0 0 0"/>
-      <xacro:wheel_geometry />
-      <material name="red"/>
-    </visual>
-  </link>
-   <link name="link_left_wheel">
-    <xacro:default_inertial mass="0.2"/>
-    <collision name="link_left_wheel_collision">
-      <origin rpy="0 1.5707 1.5707" xyz="0 0 0"/>
-      <xacro:wheel_geometry />
-    </collision>
-    <visual name="link_left_wheel_visual">
-      <origin rpy="0 1.5707 1.5707" xyz="0 0 0"/>
-      <xacro:wheel_geometry />
-      <material name="red"/>
-    </visual>
-  </link>
-  <joint name="joint_right_wheel" type="continuous">
-    <origin rpy="0 0 0" xyz="-0.05 0.15 0"/>
-    <child link="link_right_wheel"/>
-    <parent link="link_chassis"/>
-    <axis rpy="0 0 0" xyz="0 1 0"/>
-    <limit effort="10000" velocity="1000"/>
-    <joint_properties damping="1.0" friction="1.0"/>
-  </joint>
-  <joint name="joint_left_wheel" type="continuous">
-    <origin rpy="0 0 0" xyz="-0.05 -0.15 0"/>
-    <child link="link_left_wheel"/>
-    <parent link="link_chassis"/>
-    <axis rpy="0 0 0" xyz="0 1 0"/>
-    <limit effort="10000" velocity="1000"/>
-    <joint_properties damping="1.0" friction="1.0"/>
-  </joint>
+  <!-- Wheel Creation -->
+  <xacro:link_wheel name="link_right_wheel" />
+  <xacro:link_wheel name="link_left_wheel" />
+  <xacro:joint_wheel name="joint_right_wheel"  child="link_right_wheel"  origin_xyz="-0.05 0.15 0"  />
+  <xacro:joint_wheel name="joint_left_wheel"   child="link_left_wheel"   origin_xyz="-0.05 -0.15 0"  />
   <!--arm definition -->
   <link name="arm_base_link">
@@ -163,8 +140,11 @@
   <joint name="arm_joint_01" type="continuous">
   	<axis xyz="0 0 1"/>
+  	<!-- <limit effort="1000.0" velocity="1000"/>
+    <joint_properties damping="1.0" friction="1.0"/> -->
   	<origin rpy="0 0 0" xyz="0 0 0.09"/>
   	<parent link="arm_base_link"/>
   	<child link="arm_link_01"/>
   </joint>
+  <!-- Camera -->
   <link name="camera_link">
 	    <collision>
@@ -191,5 +171,5 @@
   <joint name="camera_joint" type="fixed">
 	    <axis xyz="0 1 0" />
-	    <origin xyz="0.0 0 0.0" rpy="0 0 0"/>
+	    <origin xyz="0.03 0 0.0" rpy="0 0 0"/>
 	    <parent link="arm_link_01"/>
 	    <child link="camera_link"/>
